File: placaAmplificadora/placaAmplificadora.kicad_sch (KiCad schematic)
At the start: 49 parts, among them J1 Screw_Terminal_01x03, J2 Conn_01x12_Female, J3 Conn_01x12_Female, J4 Conn_01x01_Female, J5 Conn_01x01_Female, U1 LM324, U2 AD620, U3 LM358

Commit message: kk
Parts:
- gave numbers to parts that had none: 1
- renumbered C7 to C3, C3 to C4, C8 to C5, C9 to C6, C4 to C7, C6 to C8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
