File: placaAmplificadora/placaAmplificadora.kicad_pcb (KiCad board)
At the start: 2 copper layers, 48 parts, among them J1 Screw_Terminal_01x03, J2 Conn_01x12_Female, J3 Conn_01x12_Female, J4 Conn_01x01_Female, J5 Conn_01x01_Female, J6 Conn_01x01_Female, U1 LM324, U2 LM358, U3 AD620

Commit message: sc
Routing:
- net /HPF2: track 60.1 -> 79.6 mm
- net Net-(C10-Pad1): track 54.6 -> 58.8 mm
- net Net-(C12-Pad1): track 3.30 -> 7.41 mm
- added copper zone on B.Cu, net GND
- added copper zone on F.Cu, net GND
Changed lines of the file:
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@@
   (segment (start 94.0308 103.378) (end 85.5472 103.378) (width 1) (layer "F.Cu") (net 10))
   (via (at 76.5556 91.9988) (size 0.8) (drill 0.4) (layers "F.Cu" "B.Cu") (net 10))
-  (segment (start 98.338 103.054) (end 103.3422 98.0498) (width 1) (layer "B.Cu") (net 10))
-  (segment (start 98.338 104.0892) (end 98.338 103.054) (width 1) (layer "B.Cu") (net 10))
+  (segment (start 103.3422 98.0498) (end 103.3422 95.8238) (width 1) (layer "B.Cu") (net 10))
+  (segment (start 103.0282 95.5098) (end 100.8022 95.5098) (width 1) (layer "B.Cu") (net 10))
+  (segment (start 98.338 104.0892) (end 98.3488 104.0784) (width 1) (layer "B.Cu") (net 10))
+  (segment (start 98.3488 104.0784) (end 98.3488 101.1936) (width 1) (layer "B.Cu") (net 10))
+  (segment (start 103.3422 95.8238) (end 103.0282 95.5098) (width 1) (layer "B.Cu") (net 10))
   (segment (start 76.5556 91.9988) (end 76.5556 92.9132) (width 1) (layer "B.Cu") (net 10))
-  (segment (start 103.3422 98.0498) (end 100.8022 95.5098) (width 1) (layer "B.Cu") (net 10))
+  (segment (start 98.3488 101.1936) (end 103.3422 101.1936) (width 1) (layer "B.Cu") (net 10))
   (segment (start 76.5556 92.9132) (end 71.9328 92.9132) (width 1) (layer "B.Cu") (net 10))
+  (segment (start 103.3422 101.1936) (end 103.3422 98.0498) (width 1) (layer "B.Cu") (net 10))
   (segment (start 103.338 101.1536) (end 94.1216 101.1536) (width 1) (layer "F.Cu") (net 11))
   (segment (start 103.338 104.0892) (end 103.338 101.1536) (width 1) (layer "F.Cu") (net 11))
@@
   (segment (start 94.1324 101.1428) (end 94.1324 95.3516) (width 1) (layer "F.Cu") (net 11))
   (segment (start 94.1324 110.3884) (end 94.1324 108.5596) (width 1) (layer "B.Cu") (net 11))
+  (segment (start 91.6432 110.3884) (end 91.4908 110.5408) (width 1) (layer "B.Cu") (net 11))
   (segment (start 94.0816 90.3732) (end 71.9328 90.3732) (width 1) (layer "B.Cu") (net 11))
   (segment (start 103.3272 107.696) (end 103.338 107.6852) (width 1) (layer "B.Cu") (net 11))
+  (segment (start 91.4908 110.5408) (end 91.4908 124.6016) (width 1) (layer "B.Cu") (net 11))
+  (segment (start 94.1324 110.3884) (end 91.6432 110.3884) (width 1) (layer "B.Cu") (net 11))
   (segment (start 103.338 107.6852) (end 103.338 104.0892) (width 1) (layer "B.Cu") (net 11))
   (segment (start 94.1324 95.3516) (end 94.1324 90.424) (width 1) (layer "B.Cu") (net 11))
   (segment (start 94.996 107.696) (end 103.3272 107.696) (width 1) (layer "B.Cu") (net 11))
   (segment (start 94.1324 90.424) (end 94.0816 90.3732) (width 1) (layer "B.Cu") (net 11))
+  (segment (start 91.4908 124.6016) (end 94.1832 124.6016) (width 1) (layer "B.Cu") (net 11))
   (segment (start 94.1324 108.5596) (end 94.996 107.696) (width 1) (layer "B.Cu") (net 11))
   (segment (start 100.7872 129.6016) (end 100.7872 127.3556) (width 1) (layer "F.Cu") (net 12))
@@
   (segment (start 94.1832 127.7112) (end 94.5388 127.3556) (width 1) (layer "F.Cu") (net 12))
   (segment (start 94.1832 129.6016) (end 94.1832 127.7112) (width 1) (layer "F.Cu") (net 12))
+  (segment (start 97.4852 124.6016) (end 97.4852 120.4976) (width 1) (layer "B.Cu") (net 13))
   (segment (start 97.4852 120.4976) (end 100.7872 120.4976) (width 1) (layer "B.Cu") (net 13))
   (segment (start 104.2416 124.0028) (end 104.2416 120.5484) (width 1) (layer "B.Cu") (net 14))
@@
   (segment (start 97.4852 111.8616) (end 97.4852 110.3376) (width 1) (layer "B.Cu") (net 56))
   (segment (start 94.1324 115.2144) (end 97.4852 111.8616) (width 1) (layer "B.Cu") (net 56))
+  (zone (net 4) (net_name "GND") (layers F&B.Cu) (hatch edge 0.508)
+    (connect_pads (clearance 1))
+    (min_thickness 0.254) (filled_areas_thickness no)
+    (fill yes (thermal_gap 0.508) (thermal_bridge_width 0.508) (island_removal_mode 1) (island_area_min 0))
+    (polygon
+      (pts
+        (xy 121.9708 149.352)
+        (xy 20.0152 149.3012)
+        (xy 20.0152 75.5904)
+        (xy 121.9708 75.5904)
+      )
+    )
+  )
 )
